Commit message: package elnevezés javítva a nav2.launch.py-ban mecanum.xacro-hoz explicit módon ki lettek fejtve a kerék jointok és gazebo színek

File: urdf/mecanum.xacro (robot description, xacro)
@@ -2,5 +2,5 @@
 <robot xmlns:xacro="https://www.ros.org/wiki/xacro" name="mecanum">
 <!-- <xacro:include filename="hokuyo_ust10.xacro" /> -->
-<xacro:property name="radius" value="0.05" />
+<xacro:property name="radius" value="0.065" />
 <xacro:property name="length" value="0.08" />
 <xacro:property name="box_length" value="0.5" />
@@ -41,5 +41,5 @@
     <parent link="base_link" />
     <child link="front_right_wheel" />
-    <origin xyz="0.2 -${box_width/2+length/2} -0.05" />
+    <origin xyz="0.2 -${box_width/2+length/2} -0.03" />
     <axis xyz="0 1 0" />
 </joint>
@@ -66,5 +66,5 @@
     <parent link="base_link" />
     <child link="front_left_wheel" />
-    <origin xyz="0.2 ${box_width/2+length/2} -0.05" />
+    <origin xyz="0.2 ${box_width/2+length/2} -0.03" />
     <axis xyz="0 1 0" />
 </joint>
@@ -91,5 +91,5 @@
     <parent link="base_link" />
     <child link="rear_left_wheel" />
-    <origin xyz="-0.2 ${box_width/2+length/2} -0.05" />
+    <origin xyz="-0.2 ${box_width/2+length/2} -0.03" />
     <axis xyz="0 1 0" />
 </joint>
@@ -116,9 +116,10 @@
     <parent link="base_link" />
     <child link="rear_right_wheel" />
-    <origin xyz="-0.2 -${box_width/2+length/2} -0.05" />
+    <origin xyz="-0.2 -${box_width/2+length/2} -0.03" />
     <axis xyz="0 1 0" />
 </joint>
 <link name="base_link">
     <visual>
+    <origin xyz="0 0 0" rpy="0 0 0"  />
         <geometry>
             <box size="${box_length} ${box_width} ${box_height}" />
@@ -127,5 +128,5 @@
     </visual>
     <collision>
-        <origin xyz="-0.02 0 0.035" rpy="0 0 0"  />
+        <origin xyz="0 0 0" rpy="0 0 0"  />
         <geometry>
             <box size="${box_length} ${box_width} ${box_height}" />
@@ -230,3 +231,46 @@
     </plugin>
 </gazebo>
+<gazebo reference="front_right_wheel">
+    <mu1>0.5</mu1>
+    <mu2>0.5</mu2>
+    <kp>500000.0</kp>
+    <kd>10.0</kd>
+    <maxVel>0.5</maxVel>
+    <minDepth>0.001</minDepth>
+    <fdir1>1 0 0</fdir1>
+    <material>Gazebo/Black</material>
+</gazebo>
+<gazebo reference="front_left_wheel">
+    <mu1>0.5</mu1>
+    <mu2>0.5</mu2>
+    <kp>500000.0</kp>
+    <kd>10.0</kd>
+    <maxVel>0.5</maxVel>
+    <minDepth>0.001</minDepth>
+    <fdir1>1 0 0</fdir1>
+    <material>Gazebo/Black</material>
+  </gazebo>
+  <gazebo reference="rear_right_wheel">
+    <mu1>0.5</mu1>
+    <mu2>0.5</mu2>
+    <kp>500000.0</kp>
+    <kd>10.0</kd>
+    <maxVel>0.5</maxVel>
+    <minDepth>0.001</minDepth>
+    <fdir1>1 0 0</fdir1>
+    <material>Gazebo/Black</material>
+  </gazebo>
+  <gazebo reference="rear_left_wheel">
+    <mu1>0.5</mu1>
+    <mu2>0.5</mu2>
+    <kp>500000.0</kp>
+    <kd>10.0</kd>
+    <maxVel>0.5</maxVel>
+    <minDepth>0.001</minDepth>
+    <fdir1>1 0 0</fdir1>
+    <material>Gazebo/Black</material>
+  </gazebo>
+  <gazebo reference="base_link">
+    <material>Gazebo/Yellow</material>
+  </gazebo>
 </robot>

Commit message: mu, mu2 állitgatás, fdir-ek elvileg jók

File: urdf/mecanum.xacro (robot description, xacro)
@@ -135,6 +135,6 @@
     <inertial>
         <origin xyz="-0.02 0 0.035" rpy="0 0 0" />
-        <mass value="1.0" />
-        <inertia ixx="0.00129283" ixy="0" ixz="0" iyy="0.00440742" iyz="0" izz="0.00495208" />
+        <mass value="3.0" />
+        <inertia ixx="0.025" ixy="0" ixz="0" iyy="0.065" iyz="0" izz="0.0185" />
     </inertial>
 </link>
@@ -234,7 +234,15 @@
 </gazebo>
 <gazebo reference="front_right_wheel">
-    <mu1>10.0</mu1>
-    <mu2>0.0</mu2>
-    <!-- <fdir1> 1 1 0</fdir1> -->
+    <collision>
+        <surface>
+            <friction>
+                <ode>
+                    <mu>1.5</mu>
+                    <mu2>0</mu2>
+                    <fdir1>1 1 0</fdir1>
+                </ode>
+            </friction>
+        </surface>
+    </collision>
     <kp>500000.0</kp>
     <kd>10.0</kd>
@@ -244,7 +252,15 @@
 </gazebo>
 <gazebo reference="front_left_wheel">
-    <mu1>10.0</mu1>
-    <mu2>0</mu2>
-    <!-- <fdir1> -1 1 0</fdir1> -->
+    <collision>
+        <surface>
+            <friction>
+                <ode>
+                    <mu>1.5</mu>
+                    <mu2>0.000</mu2>
+                    <fdir1>1 -1 0</fdir1>
+                </ode>
+            </friction>
+        </surface>
+    </collision>
     <kp>500000.0</kp>
     <kd>10.0</kd>
@@ -254,7 +270,15 @@
   </gazebo>
   <gazebo reference="rear_right_wheel">
-    <mu1>10.0</mu1>
-    <mu2>0.0</mu2>
-    <!-- <fdir1> -1 1 0</fdir1> -->
+    <collision>
+        <surface>
+            <friction>
+                <ode>
+                    <mu>1.5</mu>
+                    <mu2>0</mu2>
+                    <fdir1>1 -1 0</fdir1>
+                </ode>
+            </friction>
+        </surface>
+    </collision>
     <kp>500000.0</kp>
     <kd>10.0</kd>
@@ -264,7 +288,15 @@
   </gazebo>
   <gazebo reference="rear_left_wheel">
-    <mu1>10.0</mu1>
-    <mu2>0.0</mu2>
-    <fdir1> 1 0 0</fdir1>
+    <collision>
+        <surface>
+            <friction>
+                <ode>
+                    <mu>1.5</mu>
+                    <mu2>0</mu2>
+                    <fdir1>1 1 0</fdir1>
+                </ode>
+            </friction>
+        </surface>
+    </collision>
     <kp>500000.0</kp>
     <kd>10.0</kd>

Commit message: Gazebo-ban jól mozog a robot x,y és z tengely körül is, még nincs lidar plugin, RVIZ-ben nincs navigáció, LaserScan

File: urdf/mecanum.xacro (robot description, xacro)
@@ -1,4 +1,4 @@
 <?xml version="1.0"?>
-<robot xmlns:xacro="https://www.ros.org/wiki/xacro" name="mecanum">
+<robot xmlns:xacro="https://www.ros.org/wiki/xacro" name="mecanum" xmlns:ignition="http://gazebosim.org/schema">
 <!-- <xacro:include filename="hokuyo_ust10.xacro" /> -->
 <xacro:property name="radius" value="0.065" />
@@ -23,5 +23,5 @@
         <origin xyz="0 0 0" rpy="1.57075 0 0"  />
         <geometry>
-            <mesh filename="file://$(find mecanum_custom)/meshes/Mecanum_jo.stl" scale="0.0015 0.0015 0.0015" />
+            <mesh filename="file://$(find mecanum_simulation)/meshes/Mecanum_jo.stl" scale="0.0015 0.0015 0.0015" />
         </geometry>
         <material name="black" />
@@ -48,5 +48,5 @@
         <origin xyz="0 0 0" rpy="1.57075 0 0"  />
         <geometry>
-            <mesh filename="file://$(find mecanum_custom)/meshes/Mecanum_jo.stl" scale="0.0015 0.0015 0.0015" />
+            <mesh filename="file://$(find mecanum_simulation)/meshes/Mecanum_jo.stl" scale="0.0015 0.0015 0.0015" />
         </geometry>
         <material name="black" />
@@ -73,5 +73,5 @@
         <origin xyz="0 0 0" rpy="1.57075 0 0"  />
         <geometry>
-            <mesh filename="file://$(find mecanum_custom)/meshes/Mecanum_jo.stl" scale="0.0015 0.0015 0.0015" />
+            <mesh filename="file://$(find mecanum_simulation)/meshes/Mecanum_jo.stl" scale="0.0015 0.0015 0.0015" />
         </geometry>
         <material name="black" />
@@ -98,5 +98,5 @@
         <origin xyz="0 0 0" rpy="1.57075 0 0"  />
         <geometry>
-            <mesh filename="file://$(find mecanum_custom)/meshes/Mecanum_jo.stl" scale="0.0015 0.0015 0.0015" />
+            <mesh filename="file://$(find mecanum_simulation)/meshes/Mecanum_jo.stl" scale="0.0015 0.0015 0.0015" />
         </geometry>
         <material name="black" />
@@ -135,6 +135,6 @@
     <inertial>
         <origin xyz="-0.02 0 0.035" rpy="0 0 0" />
-        <mass value="3.0" />
-        <inertia ixx="0.025" ixy="0" ixz="0" iyy="0.065" iyz="0" izz="0.0185" />
+        <mass value="15.0" />
+        <inertia ixx="0.0625" ixy="0" ixz="0" iyy="0.2125" iyz="0" izz="0.25" />
     </inertial>
 </link>
@@ -147,7 +147,7 @@
 <link name="base_scan">
     <visual>
-        <origin xyz="0 0 -0.05" rpy="0 0 0"  />
-        <geometry>
-            <mesh filename="file://$(find mecanum_custom)/meshes/sensors/hokuyo_ust10.stl" scale="1 1 1" />
+        <origin xyz="0 0 -0.05" rpy="0 0 3.14"  />
+        <geometry>
+            <mesh filename="file://$(find mecanum_simulation)/meshes/sensors/hokuyo_ust10.stl" scale="1 1 1" />
         </geometry>
         <material name="white" />
@@ -208,27 +208,48 @@
 </gazebo>
 <gazebo>
-    <plugin name="nexus_ros_force_based_move" filename="libgazebo_ros_mecanum_4wd_plugin.so">
-      <robotNamespace>/</robotNamespace>
-      <commandTopic>cmd_vel</commandTopic>
-      <odometryTopic>odom</odometryTopic>
-      <odometryFrame>odom</odometryFrame>
-      <odometryRate>25.0</odometryRate>
-      <robotBaseFrame>base_footprint</robotBaseFrame>
-      <front_left_wheel_joint>front_left_wheel_joint</front_left_wheel_joint>
-      <front_right_wheel_joint>front_right_wheel_joint</front_right_wheel_joint>
-      <rear_left_wheel_joint>rear_left_wheel_joint</rear_left_wheel_joint>
-      <rear_right_wheel_joint>rear_right_wheel_joint</rear_right_wheel_joint>
-      <wheel_separation>0.34</wheel_separation>
-      <wheel_diameter>0.15</wheel_diameter>
-      <cmdVelTimeOut>0.25</cmdVelTimeOut>
-      <publishOdometryTf>true</publishOdometryTf>
+    <plugin
+      filename="libignition-gazebo-mecanum-drive-system.so"
+      name="ignition::gazebo::systems::MecanumDrive">
+      <!-- Topic for the command input -->
+      <topic>/cmd_vel</topic>
+      <!-- Wheel joints -->
+      <front_left_joint>front_left_wheel_joint</front_left_joint>
+      <front_right_joint>front_right_wheel_joint</front_right_joint>
+      <back_left_joint>rear_left_wheel_joint</back_left_joint>
+      <back_right_joint>rear_right_wheel_joint</back_right_joint>
+      <!-- Wheel parameters -->
+      <wheel_separation>0.3</wheel_separation>
+      <wheelbase>0.3</wheelbase>
+      <wheel_radius>0.1</wheel_radius>
+      <!-- Control gains and limits (optional) -->
+      <min_acceleration>-5</min_acceleration>
+      <max_acceleration>5</max_acceleration>
+      <!-- Other parameters (optional) -->
+      <odom_topic>odom</odom_topic>
+      <tf_topic>tf</tf_topic>
+      <frame_id>odom</frame_id>
+      <child_frame_id>base_footprint</child_frame_id>
+      <odom_publish_frequency>30</odom_publish_frequency>
       <publish_odom>true</publish_odom>
       <publish_odom_tf>true</publish_odom_tf>
-      <yaw_velocity_p_gain>1.0</yaw_velocity_p_gain>
-      <x_velocity_p_gain>15.0</x_velocity_p_gain>
-      <y_velocity_p_gain>15.0</y_velocity_p_gain>
-      <max_x_velocity>0.6</max_x_velocity>
-      <max_y_velocity>0.6</max_y_velocity>
-      <max_yaw_velocity>0.5</max_yaw_velocity>
+    </plugin>
+    <plugin name="ignition::gazebo::systems::OdometryPublisher" filename="libignition-gazebo-odometry-publisher-system">
+      <odom_topic>odom</odom_topic>
+      <odom_frame>odom</odom_frame>
+      <robot_base_frame>base_footprint</robot_base_frame>
+      <publish_tf>true</publish_tf>
+      <tf_topic>tf</tf_topic>
+      <odom_publish_frequency>30</odom_publish_frequency>
+      <xyz_offset>0 0 0</xyz_offset>
+      <rpy_offset>0 0 0</rpy_offset>
+    </plugin>
+    <plugin
+        filename="libignition-gazebo-joint-state-publisher-system"
+        name="ignition::gazebo::systems::JointStatePublisher">
+        <topic>joint_states</topic>
+        <joint_name>front_left_wheel_joint</joint_name>
+        <joint_name>front_right_wheel_joint</joint_name>
+        <joint_name>rear_left_wheel_joint</joint_name>
+        <joint_name>rear_right_wheel_joint</joint_name>
     </plugin>
 </gazebo>
@@ -238,7 +259,7 @@
             <friction>
                 <ode>
-                    <mu>1.5</mu>
+                    <mu1>1.5</mu1>
                     <mu2>0</mu2>
-                    <fdir1>1 1 0</fdir1>
+                    <fdir1 ignition:expressed_in="base_footprint">1 1 0</fdir1>
                 </ode>
             </friction>
@@ -246,5 +267,5 @@
     </collision>
     <kp>500000.0</kp>
-    <kd>10.0</kd>
+    <kd>100.0</kd>
     <maxVel>0.5</maxVel>
     <minDepth>0.001</minDepth>
@@ -256,7 +277,7 @@
             <friction>
                 <ode>
-                    <mu>1.5</mu>
-                    <mu2>0.000</mu2>
-                    <fdir1>1 -1 0</fdir1>
+                    <mu1>1.5</mu1>
+                    <mu2>0</mu2>
+                    <fdir1 ignition:expressed_in="base_footprint">1 -1 0</fdir1>
                 </ode>
             </friction>
@@ -264,5 +285,5 @@
     </collision>
     <kp>500000.0</kp>
-    <kd>10.0</kd>
+    <kd>100.0</kd>
     <maxVel>0.5</maxVel>
     <minDepth>0.001</minDepth>
@@ -274,7 +295,7 @@
             <friction>
                 <ode>
-                    <mu>1.5</mu>
+                    <mu1>1.5</mu1>
                     <mu2>0</mu2>
-                    <fdir1>1 -1 0</fdir1>
+                    <fdir1 ignition:expressed_in="base_footprint">1 -1 0</fdir1>
                 </ode>
             </friction>
@@ -282,5 +303,5 @@
     </collision>
     <kp>500000.0</kp>
-    <kd>10.0</kd>
+    <kd>100.0</kd>
     <maxVel>0.5</maxVel>
     <minDepth>0.001</minDepth>
@@ -292,7 +313,7 @@
             <friction>
                 <ode>
-                    <mu>1.5</mu>
+                    <mu1>1.5</mu1>
                     <mu2>0</mu2>
-                    <fdir1>1 1 0</fdir1>
+                    <fdir1 ignition:expressed_in="base_footprint">1 1 0</fdir1>
                 </ode>
             </friction>
@@ -300,5 +321,5 @@
     </collision>
     <kp>500000.0</kp>
-    <kd>10.0</kd>
+    <kd>100.0</kd>
     <maxVel>0.5</maxVel>
     <minDepth>0.001</minDepth>
@@ -307,4 +328,6 @@
   <gazebo reference="base_link">
     <material>Gazebo/Yellow</material>
+    <mu1>0.000002</mu1>
+    <mu2>0.000002</mu2>
   </gazebo>
 </robot>
